Commit message: [update]update launch file

File: xacro/OmuniRobot3.xacro (robot description, xacro)
@@ -62,5 +62,5 @@
 			<material>Gazebo/Red</material>
 			<mu1 value="0.0" />
-			<mu2 value="1.0" />
+			<mu2 value="2.0" />
 			<kp value="5000" />
 			<kd value="10" />
@@ -77,9 +77,9 @@
 		<inertial>
 			<origin xyz="0 0 0.03" rpy="0 0 0" />
-			<mass value="1.0"/>
+			<mass value="1.0"/><!--[kg]-->
 			<inertia ixx="0.001" ixy="0.0" ixz="0.0" iyy="0.001" iyz="0.0" izz="0.001"/>
 		</inertial>
 		<visual>
-			<origin xyz="0 0 0.06016" rpy="0 0 0" />
+			<origin xyz="0 0 0.0635" rpy="0 0 0" />
 			<geometry>
 				<mesh filename="package://harurobo2022/stl/3omni.stl" />
@@ -88,5 +88,5 @@
 		</visual>
 		<collision>
-			<origin xyz="0 0 0.06016" rpy="0 0 0" />
+			<origin xyz="0 0 0.0635" rpy="0 0 0" />
 			<geometry>
 				<mesh filename="package://harurobo2022/stl/3omni.stl" />
@@ -99,14 +99,14 @@
 		<mu2>0.05</mu2>
 	</gazebo>
-	<xacro:wheel_macro prefix="wheel0"  parent="base_link" xyz="-0.181 0.105 0.0635" deg="60">
+	<xacro:wheel_macro prefix="wheel0" parent="base_link" xyz="0.21 0 0.0635" deg="-90">
 		<axis xyz="0 1 0"/>
 	</xacro:wheel_macro>
-	<xacro:wheel_macro prefix="wheel1" parent="base_link" xyz="0 -0.21 0.0635" deg="0">
+	<xacro:wheel_macro prefix="wheel1"  parent="base_link" xyz="-0.105 0.181 0.0635" deg="30">
 		<axis xyz="0 1 0"/>
 	</xacro:wheel_macro>
-	<xacro:wheel_macro prefix="wheel2" parent="base_link" xyz="0.181 0.105 0.0635" deg="-60">
+	<xacro:wheel_macro prefix="wheel2" parent="base_link" xyz="-0.105 -0.181 0.0635" deg="150">
 		<axis xyz="0 1 0"/>
 	</xacro:wheel_macro>
-	<xacro:laser_macro prefix="laser" parent="base_link" xyz="0 -0.27 0.078"/>
+	<xacro:laser_macro prefix="laser" parent="base_link" xyz="0.278 0 0.078"/>
 	<xacro:imu_macro prefix="imu" parent="base_link" xyz="0.00 0 0.09"/>
 	<gazebo>

File: xacro/lidar.xacro (robot description, xacro)
@@ -4,5 +4,5 @@
 		<parent link="${parent}"/>
 		<child  link="${prefix}_link"/>
-		<origin xyz="${xyz}" rpy="0 0 0"/>
+		<origin xyz="${xyz}" rpy="0 0 ${radians(0)}"/>
 		</joint>
 		<link name="${prefix}_link">
@@ -10,5 +10,5 @@
 			<origin xyz="0 0 0" rpy="0 0 0" />
 			<geometry>
-			<cylinder radius="0.0329" length="0.04" />
+			<cylinder radius="0.021" length="0.0265" />
 			</geometry>
 			<material name="blue" />
@@ -17,5 +17,5 @@
 			<origin xyz="0 0 0" rpy="0 0 0"/>
 			<geometry>
-			<cylinder radius="0.0329" length="0.04" />
+			<cylinder radius="0.021" length="0.0265" />
 			</geometry>
 		</collision>
@@ -25,5 +25,5 @@
 		<sensor type="ray" name="${prefix}">
 			<pose>0 0 0 0 0 0</pose>
-			<visualize>false</visualize>
+			<visualize>True</visualize>
 			<update_rate>10</update_rate>
 			<ray>
@@ -32,11 +32,11 @@
 				<samples>400</samples>
 				<resolution>1</resolution>
-				<min_angle>${radians(-180)}</min_angle>
-				<max_angle>${radians(180)}</max_angle>
+				<min_angle>${radians(-120)}</min_angle>
+				<max_angle>${radians(120)}</max_angle>
 				</horizontal>
 			</scan>
 			<range>
-				<min>0.10</min>
-				<max>20.0</max>
+				<min>0.022</min>
+				<max>5.6</max>
 				<resolution>0.01</resolution>
 			</range>

Commit message: [change]changed xacro file

File: xacro/OmuniRobot3.xacro (robot description, xacro)
@@ -42,5 +42,5 @@
 			<inertial>
 				<origin xyz="0 0 0" rpy="0 0 0"/>
-				<mass value="0.02"/>
+				<mass value="0.48"/>
 				<inertia ixx="0.0001" ixy="0.0" ixz="0.0" iyy="0.0001" iyz="0.0" izz="0.0001"/>
 			</inertial>

Commit message: [change]changed mass value

File: xacro/OmuniRobot3.xacro (robot description, xacro)
@@ -42,5 +42,5 @@
 			<inertial>
 				<origin xyz="0 0 0" rpy="0 0 0"/>
-				<mass value="0.48"/>
+				<mass value="0.048"/>
 				<inertia ixx="0.0001" ixy="0.0" ixz="0.0" iyy="0.0001" iyz="0.0" izz="0.0001"/>
 			</inertial>
